File: pcb/RPi-ShieldBridge_v11.brd (EAGLE design)
At the start: 85 x 58 mm, 81 parts, among them Q1 16MHz, T1 BSS138, T2 BSS138, T3 BSS138, T4 BSS138, T5 BSS138, U1 TS5204, X1 PASSER, X2 PASSER, X3 PASSER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

Commit message: updated schematic and layout files
Parts:
- U1: value TS5204 -> TS5204-3V3
Changed lines of the file:
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@@
 <?xml version="1.0" encoding="utf-8"?>
 <!DOCTYPE eagle SYSTEM "eagle.dtd">
-<eagle version="6.5.0">
+<eagle version="6.6.0">
 <drawing>
 <settings>
@@
 <attribute name="VALUE" x="40.64" y="0.3175" size="0.8128" layer="27" font="vector"/>
 </element>
-<element name="U1" library="Voltage-Reg" package="SOT23" value="TS5204" x="44.45" y="3.175" smashed="yes">
+<element name="U1" library="Voltage-Reg" package="SOT23" value="TS5204-3V3" x="44.45" y="3.175" smashed="yes">
 <attribute name="NAME" x="43.815" y="4.9212" size="0.8128" layer="25" font="vector" ratio="10"/>
 <attribute name="VALUE" x="42.8625" y="0.3175" size="0.8128" layer="27" font="vector"/>
