File: pcb/RPi-ShieldBridge_v11.sch (EAGLE design)
At the start: 81 parts, among them Q1 16MHz, T1 BSS138, T2 BSS138, T3 BSS138, T4 BSS138, T5 BSS138, U1 TS5204, X1 PASSER, X2 PASSER, X3 PASSER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

Commit message: updated schematic and layout files
Parts:
- U1: value TS5204 -> TS5204-3V3
Changed lines of the file:
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@@
 <?xml version="1.0" encoding="utf-8"?>
 <!DOCTYPE eagle SYSTEM "eagle.dtd">
-<eagle version="6.5.0">
+<eagle version="6.6.0">
 <drawing>
 <settings>
@@
 <part name="C2" library="rcl" deviceset="C-EU" device="C0603" value="1uF"/>
 <part name="C3" library="rcl" deviceset="C-EU" device="C0603" value="1uF"/>
-<part name="U1" library="Voltage-Reg" deviceset="TS5204" device=""/>
+<part name="U1" library="Voltage-Reg" deviceset="TS5204" device="" value="TS5204-3V3"/>
 <part name="AVR" library="atmel" deviceset="MEGA8" device="-AI" value="ATmega328"/>
 <part name="GND15" library="supply1" deviceset="GND" device=""/>
