File: pcb/RPi-ShieldBridge_v11.sch (EAGLE design)
At the start: 81 parts, among them Q1 16MHz, T1 BSS138, T2 BSS138, T3 BSS138, T4 BSS138, T5 BSS138, U1 TS5204-3V3, X1 PASSER, X2 PASSER, X3 PASSER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

Commit message: cleaned up schematics and layout
Changed lines of the file:
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@@
 <setting verticaltext="up"/>
 </settings>
-<grid distance="0.1" unitdist="inch" unit="inch" style="lines" multiple="1" display="no" altdistance="0.01" altunitdist="inch" altunit="inch"/>
+<grid distance="0.05" unitdist="inch" unit="inch" style="lines" multiple="1" display="yes" altdistance="0.025" altunitdist="inch" altunit="inch"/>
 <layers>
 <layer number="1" name="Top" color="4" fill="1" visible="no" active="no"/>
@@
 <part name="U$1" library="welectronic" deviceset="WE-LOGO" device="PLACE" value="WE-LOGO"/>
 <part name="LOGO1" library="OSHW" deviceset="OSHW_LOGO_6MIL" device="X0150-NT"/>
-<part name="FRAME1" library="frames" deviceset="A4L-LOC" device=""/>
 <part name="JBL" library="jumper" deviceset="SJ" device=""/>
 <part name="T5" library="IRF-sot23" deviceset="IRLML2502" device="" value="BSS138"/>
@@
 <part name="CX" library="rcl" deviceset="C-EU" device="C0603" value="1k"/>
 <part name="C4" library="rcl" deviceset="C-EU" device="C0603" value="1uF"/>
+<part name="FRAME1" library="we-symbol" deviceset="FRAME-A4L" device=""/>
 </parts>
 <sheets>
@@
 <text x="104.14" y="6.985" size="1.27" layer="94" rot="R90">Pololu S7V7F5</text>
 <text x="171.45" y="64.77" size="3.81" layer="250">Level-Shifter</text>
-<text x="161.29" y="31.75" size="1.27" layer="95">Released under the Creative Commons Attribution Share-Alike License</text>
-<text x="161.29" y="29.21" size="1.27" layer="95">http://creativecommons.org/licenses/by-sa/4.0/</text>
-<text x="161.29" y="25.4" size="1.27" layer="95">Designed by Andreas Watterott (Watterott electronic)</text>
+<text x="162.56" y="21.59" size="1.27" layer="95">Released under the Creative Commons Attribution Share-Alike License</text>
+<text x="162.56" y="19.05" size="1.27" layer="95">http://creativecommons.org/licenses/by-sa/4.0/</text>
+<text x="162.56" y="15.24" size="1.27" layer="95">Designed by Andreas Watterott (Watterott electronic)</text>
 <text x="212.09" y="162.56" size="1.778" layer="250">Close these Jumpers for</text>
 <text x="212.09" y="160.02" size="1.778" layer="250">Arduino programming with RPi</text>
@@
 <attribute name="VALUE" x="19.177" y="151.638" size="1.778" layer="96"/>
 </instance>
-<instance part="X1" gate="G$1" x="167.64" y="17.78"/>
-<instance part="X2" gate="G$1" x="175.26" y="17.78"/>
-<instance part="X3" gate="G$1" x="182.88" y="17.78"/>
-<instance part="X4" gate="G$1" x="190.5" y="17.78"/>
-<instance part="U$1" gate="G$1" x="203.2" y="17.78"/>
-<instance part="LOGO1" gate="G$1" x="203.2" y="10.16"/>
-<instance part="FRAME1" gate="G$1" x="0" y="0" smashed="yes">
-<attribute name="DRAWING_NAME" x="217.17" y="15.24" size="2.54" layer="94" font="vector"/>
-<attribute name="LAST_DATE_TIME" x="217.17" y="10.16" size="2.286" layer="94" font="vector"/>
-<attribute name="SHEET" x="230.505" y="5.08" size="2.54" layer="94" font="vector"/>
-</instance>
+<instance part="X1" gate="G$1" x="165.1" y="7.62" smashed="yes"/>
+<instance part="X2" gate="G$1" x="170.18" y="7.62" smashed="yes"/>
+<instance part="X3" gate="G$1" x="175.26" y="7.62" smashed="yes"/>
+<instance part="X4" gate="G$1" x="180.34" y="7.62" smashed="yes"/>
+<instance part="U$1" gate="G$1" x="208.28" y="7.62"/>
+<instance part="LOGO1" gate="G$1" x="198.12" y="7.62"/>
 <instance part="JBL" gate="1" x="213.36" y="144.78" smashed="yes" rot="MR0">
 <attribute name="NAME" x="215.9" y="146.05" size="1.778" layer="95" rot="MR0"/>
@@
 <attribute name="VALUE" x="72.39" y="11.938" size="1.778" layer="96"/>
 </instance>
+<instance part="FRAME1" gate="G$1" x="0" y="0"/>
 </instances>
 <busses>
