File: hardware/RPi-ShieldBridge_v11.brd (EAGLE design)
At the start: 85 x 58 mm, 81 parts, among them Q1 16MHz, T1 BSS138, T2 BSS138, T3 BSS138, T4 BSS138, T5 BSS138, U1 TS5204-3V3, X1 PASSER, X2 PASSER, X3 PASSER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

Commit message: updated schematics
Parts:
- C1, C2, C3: value 1uF -> 2uF
Changed lines of the file:
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@@
 <?xml version="1.0" encoding="utf-8"?>
 <!DOCTYPE eagle SYSTEM "eagle.dtd">
-<eagle version="6.6.0">
+<eagle version="7.5.0">
 <drawing>
 <settings>
@@
 <layer number="51" name="tDocu" color="7" fill="1" visible="yes" active="yes"/>
 <layer number="52" name="bDocu" color="7" fill="1" visible="yes" active="yes"/>
-<layer number="53" name="tCopper" color="7" fill="11" visible="no" active="no"/>
-<layer number="54" name="bCopper" color="7" fill="1" visible="no" active="no"/>
-<layer number="56" name="wert" color="7" fill="1" visible="no" active="no"/>
 <layer number="91" name="Nets" color="2" fill="1" visible="no" active="no"/>
 <layer number="92" name="Busses" color="1" fill="1" visible="no" active="no"/>
@@
 <layer number="97" name="Info" color="7" fill="1" visible="no" active="no"/>
 <layer number="98" name="Guide" color="6" fill="1" visible="no" active="no"/>
-<layer number="100" name="Muster" color="7" fill="1" visible="no" active="no"/>
-<layer number="217" name="217bmp" color="18" fill="1" visible="no" active="no"/>
-<layer number="218" name="218bmp" color="19" fill="1" visible="no" active="no"/>
-<layer number="219" name="219bmp" color="20" fill="1" visible="no" active="no"/>
-<layer number="220" name="220bmp" color="21" fill="1" visible="no" active="no"/>
-<layer number="221" name="221bmp" color="22" fill="1" visible="no" active="no"/>
-<layer number="222" name="222bmp" color="23" fill="1" visible="no" active="no"/>
-<layer number="223" name="223bmp" color="24" fill="1" visible="no" active="no"/>
-<layer number="224" name="224bmp" color="25" fill="1" visible="no" active="no"/>
-<layer number="251" name="SMDround" color="12" fill="11" visible="no" active="no"/>
 </layers>
 <board>
@@
 <pass name="Default">
 <param name="RoutingGrid" value="50mil"/>
+<param name="AutoGrid" value="1"/>
+<param name="Efforts" value="0"/>
+<param name="TopRouterVariant" value="1"/>
 <param name="tpViaShape" value="round"/>
 <param name="PrefDir.1" value="|"/>
@@
 <attribute name="VALUE" x="59.69" y="14.9225" size="0.8128" layer="27" font="vector" rot="R180"/>
 </element>
-<element name="C2" library="rcl" package="C0603" value="1uF" x="46.99" y="3.175" smashed="yes" rot="R90">
+<element name="C2" library="rcl" package="C0603" value="2uF" x="46.99" y="3.175" smashed="yes" rot="R90">
 <attribute name="NAME" x="46.355" y="4.9213" size="0.8128" layer="25" font="vector" ratio="10"/>
 <attribute name="VALUE" x="47.3075" y="0.3175" size="0.8128" layer="27" font="vector"/>
 </element>
-<element name="C3" library="rcl" package="C0603" value="1uF" x="41.91" y="3.175" smashed="yes" rot="R90">
+<element name="C3" library="rcl" package="C0603" value="2uF" x="41.91" y="3.175" smashed="yes" rot="R90">
 <attribute name="NAME" x="41.275" y="4.9213" size="0.8128" layer="25" font="vector" ratio="10"/>
 <attribute name="VALUE" x="40.64" y="0.3175" size="0.8128" layer="27" font="vector"/>
@@
 </element>
 <element name="ARD" library="Arduino" package="UNO_ISP3" value="UNO_ISPPINS" x="8.89" y="5.08" smashed="yes"/>
-<element name="C1" library="rcl" package="C0603" value="1uF" x="49.53" y="3.175" smashed="yes" rot="R90">
+<element name="C1" library="rcl" package="C0603" value="2uF" x="49.53" y="3.175" smashed="yes" rot="R90">
 <attribute name="NAME" x="48.895" y="4.9212" size="0.8128" layer="25" font="vector" ratio="10"/>
 <attribute name="VALUE" x="49.53" y="0.3175" size="0.8128" layer="27" font="vector"/>
